Commit message: included the correct maximum speed and torque values. (set to maximum continuous values that the motors are rated at)

File: urdf/joint_params.xacro (robot description, xacro)
@@ -3,23 +3,23 @@
   <xacro:include filename="$(find dynamixel_pro_arm_description)/urdf/constants.xacro" />
   <xacro:macro name="joint1_limits">
-    <limit effort="1000.0" lower="${-M_PI * 1.5}" upper="${M_PI * 1.5}" velocity="1"/>
+    <limit effort="39.131" lower="${-M_PI * 1.5}" upper="${M_PI * 1.5}" velocity="2.5"/>
   </xacro:macro>
   <xacro:macro name="joint2_limits">
-    <limit effort="1000.0" lower="-1.7" upper="1.85" velocity="1"/>
+    <limit effort="39.131" lower="-1.7" upper="1.85" velocity="2.5"/>
   </xacro:macro>
   <property name="joint2_yaw_adjust" value="0.55"/>
   <xacro:macro name="joint3_limits">
-    <limit effort="1000.0" lower="${-M_PI }" upper="${M_PI}" velocity="1"/>
+    <limit effort="39.131" lower="${-M_PI }" upper="${M_PI}" velocity="2.5"/>
   </xacro:macro>
   <xacro:macro name="joint4_limits">
-    <limit effort="1000.0" lower="${-1.8 * 1.3}" upper="${1 * 1.3}" velocity="0.5"/>
+    <limit effort="21.142" lower="${-1.8 * 1.3}" upper="${1 * 1.3}" velocity="2.5"/>
   </xacro:macro>
   <property name="joint4_yaw_adjust" value="-0.6"/>
   <xacro:macro name="joint5_limits">
-    <limit effort="1000.0" lower="${-M_PI}" upper="${M_PI}" velocity="1.0"/>
+    <limit effort="5.596" lower="${-M_PI}" upper="${M_PI}" velocity="1.4"/>
   </xacro:macro>
   <property name="joint5_roll_adjust" value="0.55"/>
   <xacro:macro name="joint6_limits">
-    <limit effort="1000.0" lower="${-M_PI/2+5*deg2rad}" upper="${M_PI/2-5*deg2rad}" velocity="1.0"/>
+    <limit effort="5.596" lower="${-M_PI/2+5*deg2rad}" upper="${M_PI/2-5*deg2rad}" velocity="1.4"/>
   </xacro:macro>
   <property name="joint6_yaw_adjust" value="-0.65"/>
