Commit message: made the URDF a tad more gazebo friendly. It also seems that some of our inertias are so small that gazebo is rounding them to zero.

File: robots/dynamixel_pro_arm.urdf.xacro (robot description, xacro)
@@ -1,6 +1,7 @@
 <robot  name="dynamixel_pro_arm" xmlns:xacro="http://www.ros.org/wiki/xacro">
   <xacro:include filename="$(find dynamixel_pro_arm_description)/urdf/joint_params.xacro" />
-  <link
-    name="map">
+  <link name="world"/>
+  <link
+    name="base_link">
     <inertial>
       <origin
@@ -23,18 +24,22 @@
       <geometry>
         <mesh
-          filename="package://dynamixel_pro_arm_description/meshes/map.STL" />
-      </geometry>
-      <xacro:black/>
-    </visual>
-    <collision>
-      <origin
-        xyz="0 0 0"
-        rpy="0 0 0" />
-      <geometry>
-        <mesh
-          filename="package://dynamixel_pro_arm_description/meshes/map.STL" />
-      </geometry>
-    </collision>
-  </link>
+          filename="package://dynamixel_pro_arm_description/meshes/base_link.STL" />
+      </geometry>
+      <xacro:black/>
+    </visual>
+    <collision>
+      <origin
+        xyz="0 0 0"
+        rpy="0 0 0" />
+      <geometry>
+        <mesh
+          filename="package://dynamixel_pro_arm_description/meshes/base_link.STL" />
+      </geometry>
+    </collision>
+  </link>
+  <joint name="fixed" type="fixed">
+    <parent link="world"/>
+    <child link="base_link"/>
+  </joint>
   <link
     name="base1">
@@ -80,5 +85,5 @@
       rpy="-1.5707963267949 -1.04719755119659 1.5707963267949" />
     <parent
-      link="map" />
+      link="base_link" />
     <child
       link="base1" />

Commit message: removed negative intertias that were generated by the exporter. Also added damping. The arm is still unstable in gazebo.

File: robots/dynamixel_pro_arm.urdf.xacro (robot description, xacro)
@@ -15,5 +15,5 @@
         ixz="3.73992704955774E-20"
         iyy="0.00107338063659735"
-        iyz="-3.15024410056529E-06"
+        iyz="3.15024410056529E-06"
         izz="0.00136401703077675" />
     </inertial>
@@ -52,5 +52,5 @@
       <inertia
         ixx="0.000143673656725719"
-        ixy="-4.18219329301805E-06"
+        ixy="4.18219329301805E-06"
         ixz="7.91596938615036E-13"
         iyy="0.000456233710044863"
@@ -104,5 +104,5 @@
         ixz="5.05585752635912E-06"
         iyy="0.000153361641955115"
-        iyz="-1.98448185830524E-08"
+        iyz="1.98448185830524E-08"
         izz="3.04077953201017E-05" />
     </inertial>
@@ -151,6 +151,6 @@
       <inertia
         ixx="0.000553313594150257"
-        ixy="-6.59807147476319E-12"
-        ixz="-4.38331554199628E-06"
+        ixy="6.59807147476319E-12"
+        ixz="4.38331554199628E-06"
         iyy="0.000556463344423009"
         iyz="1.57596600874066E-10"
@@ -201,6 +201,6 @@
       <inertia
         ixx="0.000722720127994855"
-        ixy="-0.00069426762871192"
-        ixz="-4.11542746183462E-06"
+        ixy="0.00069426762871192"
+        ixz="4.11542746183462E-06"
         iyy="0.00465558408048209"
         iyz="2.74607957044618E-06"
@@ -252,7 +252,7 @@
         ixx="0.000190456810637275"
         ixy="7.84494923674009E-06"
-        ixz="-1.25048796604412E-05"
+        ixz="1.25048796604412E-05"
         iyy="0.000740511842342998"
-        iyz="-1.8210382605044E-06"
+        iyz="1.8210382605044E-06"
         izz="0.000658316180066946" />
     </inertial>
@@ -301,8 +301,8 @@
       <inertia
         ixx="0.000101816051726741"
-        ixy="1.67402255048959E-12"
-        ixz="-7.17181162394316E-07"
+        ixy="0.000101816051726741"
+        ixz="7.17181162394316E-07"
         iyy="0.000103434698784475"
-        iyz="-8.06089586271756E-11"
+        iyz="8.06089586271756E-11"
         izz="4.30375262150159E-05" />
     </inertial>
@@ -351,6 +351,6 @@
       <inertia
         ixx="5.91211534512154E-05"
-        ixy="-8.77944300666587E-08"
-        ixz="-1.92531044216403E-06"
+        ixy="8.77944300666587E-08"
+        ixz="1.92531044216403E-06"
         iyy="5.67480925087134E-05"
         iyz="2.07067535243446E-08"

File: urdf/constants.xacro (robot description, xacro)
@@ -1,4 +1,5 @@
 <?xml version="1.0"?>
 <robot name="dynamixel_pro_arm" xmlns:xacro="http://www.ros.org/wiki/xacro">
+  <property name="DAMPING" value="0.3"/>
   <property name="M_PI" value="3.1415926535897931" />
   <property name="M_PI_2" value="1.57079632679" />

File: urdf/joint_params.xacro (robot description, xacro)
@@ -4,22 +4,28 @@
   <xacro:macro name="joint1_limits">
     <limit effort="39.131" lower="${-M_PI * 1.5}" upper="${M_PI * 1.5}" velocity="2.5"/>
+    <dynamics damping="${DAMPING}"/>
   </xacro:macro>
   <xacro:macro name="joint2_limits">
     <limit effort="39.131" lower="-1.7" upper="1.85" velocity="2.5"/>
+    <dynamics damping="${DAMPING}"/>
   </xacro:macro>
   <property name="joint2_yaw_adjust" value="0.55"/>
   <xacro:macro name="joint3_limits">
     <limit effort="39.131" lower="${-M_PI }" upper="${M_PI}" velocity="2.5"/>
+    <dynamics damping="${DAMPING}"/>
   </xacro:macro>
   <xacro:macro name="joint4_limits">
     <limit effort="21.142" lower="${-1.8 * 1.3}" upper="${1 * 1.3}" velocity="2.5"/>
+    <dynamics damping="${DAMPING}"/>
   </xacro:macro>
   <property name="joint4_yaw_adjust" value="-0.6"/>
   <xacro:macro name="joint5_limits">
     <limit effort="5.596" lower="${-M_PI}" upper="${M_PI}" velocity="1.4"/>
+    <dynamics damping="${DAMPING}"/>
   </xacro:macro>
   <property name="joint5_roll_adjust" value="0.55"/>
   <xacro:macro name="joint6_limits">
     <limit effort="5.596" lower="${-M_PI/2+5*deg2rad}" upper="${M_PI/2-5*deg2rad}" velocity="1.4"/>
+    <dynamics damping="${DAMPING}"/>
   </xacro:macro>
   <property name="joint6_yaw_adjust" value="-0.65"/>

Commit message: a little bit of refactoring and cleanup for release.

File: robots/dynamixel_pro_arm.urdf.xacro (robot description, xacro)
@@ -18,23 +18,4 @@
         izz="0.00136401703077675" />
     </inertial>
-    <visual>
-      <origin
-        xyz="0 0 0"
-        rpy="0 0 0" />
-      <geometry>
-        <mesh
-          filename="package://dynamixel_pro_arm_description/meshes/base_link.STL" />
-      </geometry>
-      <xacro:black/>
-    </visual>
-    <collision>
-      <origin
-        xyz="0 0 0"
-        rpy="0 0 0" />
-      <geometry>
-        <mesh
-          filename="package://dynamixel_pro_arm_description/meshes/base_link.STL" />
-      </geometry>
-    </collision>
   </link>
   <joint name="fixed" type="fixed">
@@ -43,5 +24,5 @@
   </joint>
   <link
-    name="base1">
+    name="link1">
     <inertial>
       <origin
@@ -64,15 +45,15 @@
       <geometry>
         <mesh
-          filename="package://dynamixel_pro_arm_description/meshes/base1.STL" />
-      </geometry>
-      <xacro:black/>
-    </visual>
-    <collision>
-      <origin
-        xyz="0 0 0"
-        rpy="0 0 0" />
-      <geometry>
-        <mesh
-          filename="package://dynamixel_pro_arm_description/meshes/base1.STL" />
+          filename="package://dynamixel_pro_arm_description/meshes/link1.STL" />
+      </geometry>
+      <xacro:black/>
+    </visual>
+    <collision>
+      <origin
+        xyz="0 0 0"
+        rpy="0 0 0" />
+      <geometry>
+        <mesh
+          filename="package://dynamixel_pro_arm_description/meshes/link1.STL" />
       </geometry>
     </collision>
@@ -87,10 +68,10 @@
       link="base_link" />
     <child
-      link="base1" />
+      link="link1" />
     <axis
       xyz="0 0 0" />
   </joint>
   <link
-    name="base2">
+    name="link2">
     <inertial>
       <origin
@@ -113,15 +94,15 @@
       <geometry>
         <mesh
-          filename="package://dynamixel_pro_arm_description/meshes/base2.STL" />
-      </geometry>
-      <xacro:black/>
-    </visual>
-    <collision>
-      <origin
-        xyz="0 0 0"
-        rpy="0 0 0" />
-      <geometry>
-        <mesh
-          filename="package://dynamixel_pro_arm_description/meshes/base2.STL" />
+          filename="package://dynamixel_pro_arm_description/meshes/link2.STL" />
+      </geometry>
+      <xacro:black/>
+    </visual>
+    <collision>
+      <origin
+        xyz="0 0 0"
+        rpy="0 0 0" />
+      <geometry>
+        <mesh
+          filename="package://dynamixel_pro_arm_description/meshes/link2.STL" />
       </geometry>
     </collision>
@@ -134,7 +115,7 @@
       rpy="0.000329950722368627 -3.91151844547536E-19 1.16573417585641E-15" />
     <parent
-      link="base1" />
-    <child
-      link="base2" />
+      link="link1" />
+    <child
+      link="link2" />
     <axis
       xyz="1 0 0" />
@@ -142,5 +123,5 @@
   </joint>
   <link
-    name="base3">
+    name="link3">
     <inertial>
       <origin
@@ -163,15 +144,15 @@
       <geometry>
         <mesh
-          filename="package://dynamixel_pro_arm_description/meshes/base3.STL" />
-      </geometry>
-      <xacro:black/>
-    </visual>
-    <collision>
-      <origin
-        xyz="0 0 0"
-        rpy="0 0 0" />
-      <geometry>
-        <mesh
-          filename="package://dynamixel_pro_arm_description/meshes/base3.STL" />
+          filename="package://dynamixel_pro_arm_description/meshes/link3.STL" />
+      </geometry>
+      <xacro:black/>
+    </visual>
+    <collision>
+      <origin
+        xyz="0 0 0"
+        rpy="0 0 0" />
+      <geometry>
+        <mesh
+          filename="package://dynamixel_pro_arm_description/meshes/link3.STL" />
       </geometry>
     </collision>
@@ -184,7 +165,7 @@
       rpy="1.07672117749535E-15 -3.33077071782914E-16 ${joint2_yaw_adjust -0.448514927738314}" />
     <parent
-      link="base2" />
-    <child
-      link="base3" />
+      link="link2" />
+    <child
+      link="link3" />
     <axis
       xyz="0 0 1" />
@@ -192,5 +173,5 @@
   </joint>
   <link
-    name="base4">
+    name="link4">
     <inertial>
       <origin
@@ -213,15 +194,15 @@
       <geometry>
         <mesh
-          filename="package://dynamixel_pro_arm_description/meshes/base4.STL" />
-      </geometry>
-      <xacro:black/>
-    </visual>
-    <collision>
-      <origin
-        xyz="0 0 0"
-        rpy="0 0 0" />
-      <geometry>
-        <mesh
-          filename="package://dynamixel_pro_arm_description/meshes/base4.STL" />
+          filename="package://dynamixel_pro_arm_description/meshes/link4.STL" />
+      </geometry>
+      <xacro:black/>
+    </visual>
+    <collision>
+      <origin
+        xyz="0 0 0"
+        rpy="0 0 0" />
+      <geometry>
+        <mesh
+          filename="package://dynamixel_pro_arm_description/meshes/link4.STL" />
       </geometry>
     </collision>
@@ -234,7 +215,7 @@
       rpy="3.05278468838634 -1.03419334727961E-16 -6.84174938925253E-15" />
     <parent
-      link="base3" />
-    <child
-      link="base4" />
+      link="link3" />
+    <child
+      link="link4" />
     <axis
       xyz="1 0 0" />
@@ -242,5 +223,5 @@
   </joint>
   <link
-    name="base5">
+    name="link5">
     <inertial>
       <origin
@@ -263,15 +244,15 @@
       <geometry>
         <mesh
-          filename="package://dynamixel_pro_arm_description/meshes/base5.STL" />
-      </geometry>
-      <xacro:black/>
-    </visual>
-    <collision>
-      <origin
-        xyz="0 0 0"
-        rpy="0 0 0" />
-      <geometry>
-        <mesh
-          filename="package://dynamixel_pro_arm_description/meshes/base5.STL" />
+          filename="package://dynamixel_pro_arm_description/meshes/link5.STL" />
+      </geometry>
+      <xacro:black/>
+    </visual>
+    <collision>
+      <origin
+        xyz="0 0 0"
+        rpy="0 0 0" />
+      <geometry>
+        <mesh
+          filename="package://dynamixel_pro_arm_description/meshes/link5.STL" />
       </geometry>
     </collision>
@@ -284,7 +265,7 @@
       rpy="-1.80411241501588E-16 6.24500451351651E-17 ${joint4_yaw_adjust + -0.166489329587427}" />
     <parent
-      link="base4" />
-    <child
-      link="base5" />
+      link="link4" />
+    <child
+      link="link5" />
     <axis
       xyz="0 0 1" />
@@ -292,5 +273,5 @@
   </joint>
   <link
-    name="base6">
+    name="link6">
     <inertial>
       <origin
@@ -313,15 +294,15 @@
       <geometry>
         <mesh
-          filename="package://dynamixel_pro_arm_description/meshes/base6.STL" />
-      </geometry>
-      <xacro:black/>
-    </visual>
-    <collision>
-      <origin
-        xyz="0 0 0"
-        rpy="0 0 0" />
-      <geometry>
-        <mesh
-          filename="package://dynamixel_pro_arm_description/meshes/base6.STL" />
+          filename="package://dynamixel_pro_arm_description/meshes/link6.STL" />
+      </geometry>
+      <xacro:black/>
+    </visual>
+    <collision>
+      <origin
+        xyz="0 0 0"
+        rpy="0 0 0" />
+      <geometry>
+        <mesh
+          filename="package://dynamixel_pro_arm_description/meshes/link6.STL" />
       </geometry>
     </collision>
@@ -334,7 +315,7 @@
       rpy="${joint5_roll_adjust + -0.486056396438146} -2.4980018054066E-16 2.38697950294409E-15" />
     <parent
-      link="base5" />
-    <child
-      link="base6" />
+      link="link5" />
+    <child
+      link="link6" />
     <axis
       xyz="1 0 0" />
@@ -342,5 +323,5 @@
   </joint>
   <link
-    name="base7">
+    name="link7">
     <inertial>
       <origin
@@ -363,15 +344,15 @@
       <geometry>
         <mesh
-          filename="package://dynamixel_pro_arm_description/meshes/base7.STL" />
-      </geometry>
-      <xacro:black/>
-    </visual>
-    <collision>
-      <origin
-        xyz="0 0 0"
-        rpy="0 0 0" />
-      <geometry>
-        <mesh
-          filename="package://dynamixel_pro_arm_description/meshes/base7.STL" />
+          filename="package://dynamixel_pro_arm_description/meshes/link7.STL" />
+      </geometry>
+      <xacro:black/>
+    </visual>
+    <collision>
+      <origin
+        xyz="0 0 0"
+        rpy="0 0 0" />
+      <geometry>
+        <mesh
+          filename="package://dynamixel_pro_arm_description/meshes/link7.STL" />
       </geometry>
     </collision>
@@ -384,7 +365,7 @@
       rpy="1.60982338570648E-15 1.16573417585641E-15 ${joint6_yaw_adjust + 0.621053840565577}" />
     <parent
-      link="base6" />
-    <child
-      link="base7" />
+      link="link6" />
+    <child
+      link="link7" />
     <axis
       xyz="0 0 1" />
@@ -415,3 +396,4 @@
     <cfmDamping>1</cfmDamping>
   </gazebo>
+  <xacro:include filename="$(find dynamixel_pro_arm_description)/urdf/gazebo.xacro" />
 </robot>
